Commit message: launch  init

File: urdf/robot.urdf (robot description, URDF)
Before this commit: robot my_robot, 3 links, 2 joints
Links:
- removed link link1
- added link front_wheel_link, mass 0.1; collision cylinder length=0.08 radius=0.1; visual cylinder length=0.08 radius=0.1
- added link left_wheel_link, mass 0.1; collision cylinder length=0.1 radius=0.12; visual cylinder length=0.1 radius=0.12
- link base_link: mass None -> 1.0; geometry collision box size=0.8 0.5 0.2; visual box size=0.8 0.5 0.2
- link right_wheel_link: mass None -> 0.1; geometry collision cylinder length=0.1 radius=0.12; visual cylinder length=0.1 radius=0.12
Joints:
- removed joint joint1
- added joint front_wheel_joint: type continuous, parent base_link, child front_wheel_link, origin xyz=0.3 0 -0.1 rpy=0 1.5708 0, axis 0 1 0
- added joint left_wheel_joint: type continuous, parent base_link, child left_wheel_link, origin xyz=-0.25 -0.3 -0.12 rpy=0 1.5708 0, axis 0 1 0
- joint right_wheel_joint: origin xyz=0.5 0 0.1 rpy=0 1.57 0 -> xyz=-0.25 0.3 -0.12 rpy=0 1.5708 0
