Commit message: 将一个xacro文件拆分成丧各增加维护性

File: install/robot_description/share/robot_description/urdf/robot.xacro (robot description, xacro)
@@ -1,112 +1,7 @@
 <?xml version="1.0"?>
 <robot name="tricycle_robot" xmlns:xacro="http://www.ros.org/wiki/xacro">
-    <!-- 车身（方块） -->
-    <link name="base_link">
-        <visual>
-            <geometry>
-                <box size="0.8 0.5 0.2"/>
-            </geometry>
-            <origin xyz="0 0 0.1"/>
-            <material name="blue">
-                <color rgba="0 0 1 1"/>
-            </material>
-        </visual>
-        <collision>
-            <geometry>
-                <box size="0.8 0.5 0.2"/>
-            </geometry>
-            <origin xyz="0 0 0.1"/>
-        </collision>
-        <inertial>
-            <mass value="1.0"/>
-            <inertia ixx="0.1" ixy="0" ixz="0" iyy="0.1" iyz="0" izz="0.1"/>
-        </inertial>
-    </link>
-    <!-- 左后轮 -->
-    <link name="left_wheel_link">
-        <visual>
-            <geometry>
-                <cylinder length="0.1" radius="0.12"/>
-            </geometry>
-            <origin xyz="0 0 0" rpy="0 1.5708 0"/>
-            <material name="black">
-                <color rgba="0.1 0.1 0.1 1"/>
-            </material>
-        </visual>
-        <collision>
-            <geometry>
-                <cylinder length="0.1" radius="0.12"/>
-            </geometry>
-            <origin xyz="0 0 0" rpy="0 1.5708 0"/>
-        </collision>
-        <inertial>
-            <mass value="0.1"/>
-            <inertia ixx="0.001" ixy="0" ixz="0" iyy="0.001" iyz="0" izz="0.001"/>
-        </inertial>
-    </link>
-    <!-- 右后轮 -->
-    <link name="right_wheel_link">
-        <visual>
-            <geometry>
-                <cylinder length="0.1" radius="0.12"/>
-            </geometry>
-            <origin xyz="0 0 0" rpy="0 1.5708 0"/>
-            <material name="black">
-                <color rgba="0.1 0.1 0.1 1"/>
-            </material>
-        </visual>
-        <collision>
-            <geometry>
-                <cylinder length="0.1" radius="0.12"/>
-            </geometry>
-            <origin xyz="0 0 0" rpy="0 1.5708 0"/>
-        </collision>
-        <inertial>
-            <mass value="0.1"/>
-            <inertia ixx="0.001" ixy="0" ixz="0" iyy="0.001" iyz="0" izz="0.001"/>
-        </inertial>
-    </link>
-    <!-- 前轮 -->
-    <link name="front_wheel_link">
-        <visual>
-            <geometry>
-                <cylinder length="0.08" radius="0.1"/>
-            </geometry>
-            <origin xyz="0 0 0" rpy="0 1.5708 0"/>
-            <material name="black">
-                <color rgba="0.1 0.1 0.1 1"/>
-            </material>
-        </visual>
-        <collision>
-            <geometry>
-                <cylinder length="0.08" radius="0.1"/>
-            </geometry>
-            <origin xyz="0 0 0" rpy="0 1.5708 0"/>
-        </collision>
-        <inertial>
-            <mass value="0.1"/>
-            <inertia ixx="0.001" ixy="0" ixz="0" iyy="0.001" iyz="0" izz="0.001"/>
-        </inertial>
-    </link>
-    <!-- 左后轮关节 -->
-    <joint name="left_wheel_joint" type="continuous">
-        <parent link="base_link"/>
-        <child link="left_wheel_link"/>
-        <origin xyz="-0.25 -0.3 -0.12" rpy="0 1.5708 0"/>
-        <axis xyz="0 1 0"/>
-    </joint>
-    <!-- 右后轮关节 -->
-    <joint name="right_wheel_joint" type="continuous">
-        <parent link="base_link"/>
-        <child link="right_wheel_link"/>
-        <origin xyz="-0.25 0.3 -0.12" rpy="0 1.5708 0"/>
-        <axis xyz="0 1 0"/>
-    </joint>
-    <!-- 前轮关节 -->
-    <joint name="front_wheel_joint" type="continuous">
-        <parent link="base_link"/>
-        <child link="front_wheel_link"/>
-        <origin xyz="0.3 0 -0.1" rpy="0 1.5708 0"/>
-        <axis xyz="0 1 0"/>
-    </joint>
+    <!-- ==================== 宏定义 ==================== -->
+    <xacro:property name="PI" value="3.1415926535" />
+    <xacro:include filename="$(find robot_description)/urdf/common_property.xacro" />
+    <xacro:include filename="$(find robot_description)/urdf/mobile.xacro" />
 </robot>
