Commit message: 增加gazebo plugin

File: install/robot_description/share/robot_description/urdf/common_property.xacro (robot description, xacro)
@@ -13,3 +13,11 @@
         <color rgba="0.05 0.05 0.05 1"/>
     </material>
+    <xacro:macro name="box_inertial" params="mxyz O_xyz O_rpy">
+        <inertial>
+            <mass value="$S{mxyz[0]}"/>
+            <origin xyz="$S{O_xyz}" rpy="$S{O_rpy}"/>
+            <inertia ixx="$S{(m/12)*(y*y+z*z)}" ixy="0" ixz="0"
+            iyy="$S{(m/12)*(x*x+z*z)}" iyz="0 " izz="$S{(m/12)*(x*x+y*y)}"/>
+        </inertial>
+    </xacro:macro>
 </robot>
